File: docs/cyclonev-diagram/ALM.kicad_sch (KiCad schematic)
At the start: 54 parts

Commit message: Clock mux documentation
Connections:
- net C: now also U?. (E1); no longer U?. (TS)
- net D: now also U?. (TS); no longer U?. (E1)
- new net: A.3, U?. (S), U?. (TS)
- new net: U?. (E1), U?. (S1)
- new net: U?. (S1), U?. (TS)
- new net: TCLR_SEL. (O), U?.~ (R), U?.~ (R)
- new net: TCLK_SEL. (O), U?.~ (R), U?.~ (R)
- new net: BCLK_SEL. (O), U?.~ (R), U?.~ (R)
- new net: U?.~ (SO), U?.~ (SO)
- new net: BCLR_SEL. (O), U?.~ (R), U?.~ (R)
Changed lines of the file:
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@@
     (effects (font (size 1.27 1.27)) (justify right))
   )
-  (hierarchical_label "D" (shape input) (at 6.35 66.04 180)
+  (hierarchical_label "C" (shape input) (at 6.35 66.04 180)
     (effects (font (size 1.27 1.27)) (justify right))
   )
@@
     (effects (font (size 1.27 1.27)) (justify right))
   )
-  (hierarchical_label "C" (shape input) (at 6.35 39.37 180)
+  (hierarchical_label "D" (shape input) (at 6.35 39.37 180)
     (effects (font (size 1.27 1.27)) (justify right))
   )
